Commit message: Created core URDF

File: description/colors.xacro (robot description, xacro)
@@ -4,5 +4,5 @@
 	<material name="black">
 		<color rgba="0.0 0.0 0.0 1.0" />
-    </material>
+	</material>
 	<material name="red">
 		<color rgba="0.7 0.0 0.0 1.0"/>

File: description/robot.urdf.xacro (robot description, xacro)
@@ -1,4 +1,5 @@
 <?xml version="1.0"?>
 <robot xmlns:xacro="http://www.ros.org/wiki/xacro" name="robot">
+	<xacro:include filename="inertial_macros.xacro"/>
 	<xacro:include filename="robot_core.xacro"/>
 </robot>

File: description/robot_core.xacro (robot description, xacro)
@@ -20,4 +20,13 @@
 			<material name="gray"/>
 		</visual>
+		<collision>
+			<origin xyz="0.15 0.0 0.05"/>
+			<geometry>
+				<cylinder radius="0.15" length="0.1"/>
+			</geometry>
+		</collision>
+		<xacro:inertial_cylinder mass="0.5" length="0.1" radius="0.15">
+			<origin xyz="0.15 0.0 0.05" rpy="0.0 0.0 0.0"/>
+		</xacro:inertial_cylinder>
 	</link>
 	<!-- LEFT WHEEL -->
@@ -35,4 +44,12 @@
 			<material name="black"/>
 		</visual>
+		<collision>
+			<geometry>
+				<cylinder radius="0.05" length="0.04"/>
+			</geometry>
+		</collision>
+		<xacro:inertial_cylinder mass="0.1" length="0.04" radius="0.05">
+			<origin xyz="0.0 0.0 0.0" rpy="0.0 0.0 0.0"/>
+		</xacro:inertial_cylinder>
 	</link>
 	<!-- RIGHT WHEEL -->
@@ -50,4 +67,12 @@
 			<material name="black"/>
 		</visual>
+		<collision>
+			<geometry>
+				<cylinder radius="0.05" length="0.04"/>
+			</geometry>
+		</collision>
+		<xacro:inertial_cylinder mass="0.1" length="0.04" radius="0.05">
+			<origin xyz="0.0 0.0 0.0" rpy="0.0 0.0 0.0"/>
+		</xacro:inertial_cylinder>
 	</link>
 	<!-- CASTER WHEEL -->
@@ -64,4 +89,12 @@
 			<material name="black"/>
 		</visual>
+		<collision>
+			<geometry>
+				<sphere radius="0.05"/>
+			</geometry>
+		</collision>
+		<xacro:inertial_sphere mass="0.1" radius="0.05">
+			<origin xyz="0.0 0.0 0.0" rpy="0.0 0.0 0.0"/>
+		</xacro:inertial_sphere>
 	</link>
 </robot>

Commit message: Added camera feed to sim env

File: description/colors.xacro (robot description, xacro)
@@ -1,22 +1,22 @@
 <?xml version="1.0"?>
 <robot xmlns:xacro="http://www.ros.org/wiki/xacro">
-	<!-- Colors Definition -->
-	<material name="black">
-		<color rgba="0.0 0.0 0.0 1.0" />
-	</material>
-	<material name="red">
-		<color rgba="0.7 0.0 0.0 1.0"/>
-	</material>
-	<material name="blue">
-		<color rgba="0.0 0.0 0.7 1.0"/>
-	</material>
-	<material name="green">
-		<color rgba="0.0 0.7 0.0 1.0"/>
-	</material>
-	<material name="gray">
-		<color rgba="0.5 0.5 0.6 1.0"/>
-	</material>
-	<material name="white">
-		<color rgba="1.0 1.0 1.0 1.0" />
-	</material>
+    <!-- Colors Definition -->
+    <material name="black">
+        <color rgba="0.0 0.0 0.0 1.0" />
+    </material>
+    <material name="red">
+        <color rgba="0.7 0.0 0.0 1.0"/>
+    </material>
+    <material name="blue">
+        <color rgba="0.0 0.0 0.7 1.0"/>
+    </material>
+    <material name="green">
+        <color rgba="0.0 0.7 0.0 1.0"/>
+    </material>
+    <material name="gray">
+        <color rgba="0.5 0.5 0.6 1.0"/>
+    </material>
+    <material name="white">
+        <color rgba="1.0 1.0 1.0 1.0" />
+    </material>
 </robot>

File: description/inertial_macros.xacro (robot description, xacro)
@@ -1,34 +1,34 @@
 <?xml version="1.0"?>
 <robot xmlns:xacro="http://www.ros.org/wiki/xacro">
-	<!-- Specify some standard inertial calculations https://en.wikipedia.org/wiki/List_of_moments_of_inertia -->
-	<xacro:macro name="inertial_box" params="mass x y z *origin">
-		<inertial>
-			<xacro:insert_block name="origin"/>
-			<mass value="${mass}" />
-			<inertia ixx="${(1/12) * mass * (y*y+z*z)}" ixy="0.0" ixz="0.0"
-					iyy="${(1/12) * mass * (x*x+z*z)}" iyz="0.0"
-					izz="${(1/12) * mass * (x*x+y*y)}"
-			/>
-		</inertial>
-	</xacro:macro>
-	<xacro:macro name="inertial_cylinder" params="mass length radius *origin">
-		<inertial>
-			<xacro:insert_block name="origin"/>
-			<mass value="${mass}" />
-			<inertia ixx="${(1/12) * mass * (3*radius*radius + length*length)}" ixy="0.0" ixz="0.0"
-					iyy="${(1/12) * mass * (3*radius*radius + length*length)}" iyz="0.0"
-					izz="${(1/2) * mass * (radius*radius)}"
-			/>
-		</inertial>
-	</xacro:macro>
-	<xacro:macro name="inertial_sphere" params="mass radius *origin">
-		<inertial>
-			<xacro:insert_block name="origin"/>
-			<mass value="${mass}"/>
-			<inertia ixx="${(2/5) * mass * (radius*radius)}" ixy="0.0" ixz="0.0"
-					iyy="${(2/5) * mass * (radius*radius)}" iyz="0.0"
-					izz="${(2/5) * mass * (radius*radius)}"
-			/>
-		</inertial>
-	</xacro:macro>
+    <!-- Specify some standard inertial calculations https://en.wikipedia.org/wiki/List_of_moments_of_inertia -->
+    <xacro:macro name="inertial_box" params="mass x y z *origin">
+        <inertial>
+            <xacro:insert_block name="origin"/>
+            <mass value="${mass}" />
+            <inertia ixx="${(1/12) * mass * (y*y+z*z)}" ixy="0.0" ixz="0.0"
+                    iyy="${(1/12) * mass * (x*x+z*z)}" iyz="0.0"
+                    izz="${(1/12) * mass * (x*x+y*y)}"
+            />
+        </inertial>
+    </xacro:macro>
+    <xacro:macro name="inertial_cylinder" params="mass length radius *origin">
+        <inertial>
+            <xacro:insert_block name="origin"/>
+            <mass value="${mass}" />
+            <inertia ixx="${(1/12) * mass * (3*radius*radius + length*length)}" ixy="0.0" ixz="0.0"
+                    iyy="${(1/12) * mass * (3*radius*radius + length*length)}" iyz="0.0"
+                    izz="${(1/2) * mass * (radius*radius)}"
+            />
+        </inertial>
+    </xacro:macro>
+    <xacro:macro name="inertial_sphere" params="mass radius *origin">
+        <inertial>
+            <xacro:insert_block name="origin"/>
+            <mass value="${mass}"/>
+            <inertia ixx="${(2/5) * mass * (radius*radius)}" ixy="0.0" ixz="0.0"
+                    iyy="${(2/5) * mass * (radius*radius)}" iyz="0.0"
+                    izz="${(2/5) * mass * (radius*radius)}"
+            />
+        </inertial>
+    </xacro:macro>
 </robot>

File: description/lidar.xacro (robot description, xacro)
@@ -1,54 +1,54 @@
 <?xml version="1.0"?>
 <robot xmlns:xacro="http://www.ros.org/wiki/xacro">
-	<joint name="lidar_joint" type="fixed">
-		<origin xyz="0.15 0.0 0.12" rpy="0.0 0.0 0.0"/>
-		<parent link="chassis"/>
-		<child link="lidar"/>
-	</joint>
-	<link name="lidar">
-		<visual>
-			<geometry>
-				<cylinder radius="0.05" length="0.04"/>
-			</geometry>
-			<material name="red"/>
-		</visual>
-		<collision>
-			<geometry>
-				<cylinder radius="0.05" length="0.04"/>
-			</geometry>
-		</collision>
-		<xacro:inertial_cylinder mass="0.1" length="0.04" radius="0.05">
-			<origin xyz="0.0 0.0 0.0" rpy="0.0 0.0 0.0"/>
-		</xacro:inertial_cylinder>
-	</link>
-	<gazebo reference="lidar">
-		<material>Gazebo/Red</material>
-		<sensor name="lidar" type="ray">
-			<pose> 0 0 0 0 0 0 </pose>
-			<visualize>true</visualize>
-			<update_rate>10</update_rate>
-			<ray>
-				<scan>
-					<horizontal>
-						<samples>360</samples>
-						<resolution>1</resolution>
-						<min_angle>-3.14</min_angle>
-						<max_angle>3.14</max_angle>
-					</horizontal>
-				</scan>
-				<range>
-					<min>0.3</min>
-					<max>12</max>
-					<resolution>0.01</resolution>
-				</range>
-			</ray>
-			<plugin name="lidar_controller" filename="libgazebo_ros_ray_sensor.so">
-				<ros>
-					<argument>~/out:=scan</argument>
-				</ros>
-				<output_type>sensor_msgs/LaserScan</output_type>
-				<frame_name>lidar</frame_name>
-			</plugin>
-		</sensor>
-	</gazebo>
+    <joint name="lidar_joint" type="fixed">
+        <origin xyz="0.15 0.0 0.12" rpy="0.0 0.0 0.0"/>
+        <parent link="chassis"/>
+        <child link="lidar"/>
+    </joint>
+    <link name="lidar">
+        <visual>
+            <geometry>
+                <cylinder radius="0.05" length="0.04"/>
+            </geometry>
+            <material name="red"/>
+        </visual>
+        <collision>
+            <geometry>
+                <cylinder radius="0.05" length="0.04"/>
+            </geometry>
+        </collision>
+        <xacro:inertial_cylinder mass="0.1" length="0.04" radius="0.05">
+            <origin xyz="0.0 0.0 0.0" rpy="0.0 0.0 0.0"/>
+        </xacro:inertial_cylinder>
+    </link>
+    <gazebo reference="lidar">
+        <material>Gazebo/Red</material>
+        <sensor name="lidar" type="ray">
+            <pose> 0 0 0 0 0 0 </pose>
+            <visualize>false</visualize>
+            <update_rate>10</update_rate>
+            <ray>
+                <scan>
+                    <horizontal>
+                        <samples>360</samples>
+                        <resolution>1</resolution>
+                        <min_angle>-3.14</min_angle>
+                        <max_angle>3.14</max_angle>
+                    </horizontal>
+                </scan>
+                <range>
+                    <min>0.3</min>
+                    <max>12</max>
+                    <resolution>0.01</resolution>
+                </range>
+            </ray>
+            <plugin name="lidar_controller" filename="libgazebo_ros_ray_sensor.so">
+                <ros>
+                    <argument>~/out:=scan</argument>
+                </ros>
+                <output_type>sensor_msgs/LaserScan</output_type>
+                <frame_name>lidar</frame_name>
+            </plugin>
+        </sensor>
+    </gazebo>
 </robot>

File: description/robot.urdf.xacro (robot description, xacro)
@@ -1,7 +1,8 @@
 <?xml version="1.0"?>
 <robot xmlns:xacro="http://www.ros.org/wiki/xacro" name="robot">
-	<xacro:include filename="inertial_macros.xacro"/>
-	<xacro:include filename="robot_core.xacro"/>
-	<xacro:include filename="gazebo_control.xacro"/>
-	<xacro:include filename="lidar.xacro"/>
+    <xacro:include filename="inertial_macros.xacro"/>
+    <xacro:include filename="robot_core.xacro"/>
+    <xacro:include filename="gazebo_control.xacro"/>
+    <xacro:include filename="lidar.xacro"/>
+    <xacro:include filename="camera.xacro"/>
 </robot>

File: description/robot_core.xacro (robot description, xacro)
@@ -1,114 +1,114 @@
 <?xml version="1.0"?>
 <robot xmlns:xacro="http://www.ros.org/wiki/xacro">
-	<xacro:include filename="colors.xacro" />
-	<!-- BASE LINK -->
-	<link name="base_link">
-	</link>
-	<!-- CHASSIS -->
-	<joint name="chassis_joint" type="fixed">
-		<parent link="base_link"/>
-		<child link="chassis"/>
-		<origin xyz="-0.15 0.0 0.0"/>
-	</joint>
-	<link name="chassis">
-		<visual>
-			<!-- origin offset (review robot dimensions) -->
-			<origin xyz="0.15 0.0 0.05"/>
-			<geometry>
-				<cylinder radius="0.15" length="0.10"/>
-			</geometry>
-			<material name="gray"/>
-		</visual>
-		<collision>
-			<origin xyz="0.15 0.0 0.05"/>
-			<geometry>
-				<cylinder radius="0.15" length="0.1"/>
-			</geometry>
-		</collision>
-		<xacro:inertial_cylinder mass="0.5" length="0.1" radius="0.15">
-			<origin xyz="0.15 0.0 0.05" rpy="0.0 0.0 0.0"/>
-		</xacro:inertial_cylinder>
-	</link>
-	<gazebo reference="chassis">
-		<material>Gazebo/LightGray</material>
-	</gazebo>
-	<!-- LEFT WHEEL -->
-	<joint name="left_wheel_joint" type="continuous">
-		<origin xyz="0.0 0.175 0.0" rpy="-${pi/2} 0.0 0.0"/>
-		<parent link="base_link"/>
-		<child link="left_wheel"/>
-		<axis xyz="0.0 0.0 1.0"/>
-	</joint>
-	<link name="left_wheel">
-		<visual>
-			<geometry>
-				<cylinder radius="0.05" length="0.04"/>
-			</geometry>
-			<material name="black"/>
-		</visual>
-		<collision>
-			<geometry>
-				<cylinder radius="0.05" length="0.04"/>
-			</geometry>
-		</collision>
-		<xacro:inertial_cylinder mass="0.1" length="0.04" radius="0.05">
-			<origin xyz="0.0 0.0 0.0" rpy="0.0 0.0 0.0"/>
-		</xacro:inertial_cylinder>
-	</link>
-	<gazebo reference="left_wheel">
-		<material>Gazebo/Black</material>
-	</gazebo>
-	<!-- RIGHT WHEEL -->
-	<joint name="right_wheel_joint" type="continuous">
-		<origin xyz="0.0 -0.175 0.0" rpy="${pi/2} 0.0 0.0"/>
-		<parent link="base_link"/>
-		<child link="right_wheel"/>
-		<axis xyz="0.0 0.0 -1.0"/>
-	</joint>
-	<link name="right_wheel">
-		<visual>
-			<geometry>
-				<cylinder radius="0.05" length="0.04"/>
-			</geometry>
-			<material name="black"/>
-		</visual>
-		<collision>
-			<geometry>
-				<cylinder radius="0.05" length="0.04"/>
-			</geometry>
-		</collision>
-		<xacro:inertial_cylinder mass="0.1" length="0.04" radius="0.05">
-			<origin xyz="0.0 0.0 0.0" rpy="0.0 0.0 0.0"/>
-		</xacro:inertial_cylinder>
-	</link>
-	<gazebo reference="right_wheel">
-		<material>Gazebo/Black</material>
-	</gazebo>
-	<!-- CASTER WHEEL -->
-	<joint name="caster_wheel_joint" type="fixed">
-		<origin xyz="0.075 0.0 0.0"/>
-		<parent link="chassis"/>
-		<child link="caster_wheel"/>
-	</joint>
-	<link name="caster_wheel">
-		<visual>
-			<geometry>
-				<sphere radius="0.05"/>
-			</geometry>
-			<material name="black"/>
-		</visual>
-		<collision>
-			<geometry>
-				<sphere radius="0.05"/>
-			</geometry>
-		</collision>
-		<xacro:inertial_sphere mass="0.5" radius="0.05">
-			<origin xyz="0.0 0.0 0.0" rpy="0.0 0.0 0.0"/>
-		</xacro:inertial_sphere>
-	</link>
-	<gazebo reference="caster_wheel">
-		<material>Gazebo/Black</material>
-		<mu1 value="0.001"/>
-		<mu2 value="0.001"/>
-	</gazebo>
+    <xacro:include filename="colors.xacro" />
+    <!-- BASE LINK -->
+    <link name="base_link">
+    </link>
+    <!-- CHASSIS -->
+    <joint name="chassis_joint" type="fixed">
+        <parent link="base_link"/>
+        <child link="chassis"/>
+        <origin xyz="-0.15 0.0 0.0"/>
+    </joint>
+    <link name="chassis">
+        <visual>
+            <!-- origin offset (review robot dimensions) -->
+            <origin xyz="0.15 0.0 0.05"/>
+            <geometry>
+                <cylinder radius="0.15" length="0.10"/>
+            </geometry>
+            <material name="gray"/>
+        </visual>
+        <collision>
+            <origin xyz="0.15 0.0 0.05"/>
+            <geometry>
+                <cylinder radius="0.15" length="0.1"/>
+            </geometry>
+        </collision>
+        <xacro:inertial_cylinder mass="0.5" length="0.1" radius="0.15">
+            <origin xyz="0.15 0.0 0.05" rpy="0.0 0.0 0.0"/>
+        </xacro:inertial_cylinder>
+    </link>
+    <gazebo reference="chassis">
+        <material>Gazebo/LightGray</material>
+    </gazebo>
+    <!-- LEFT WHEEL -->
+    <joint name="left_wheel_joint" type="continuous">
+        <origin xyz="0.0 0.175 0.0" rpy="-${pi/2} 0.0 0.0"/>
+        <parent link="base_link"/>
+        <child link="left_wheel"/>
+        <axis xyz="0.0 0.0 1.0"/>
+    </joint>
+    <link name="left_wheel">
+        <visual>
+            <geometry>
+                <cylinder radius="0.05" length="0.04"/>
+            </geometry>
+            <material name="black"/>
+        </visual>
+        <collision>
+            <geometry>
+                <cylinder radius="0.05" length="0.04"/>
+            </geometry>
+        </collision>
+        <xacro:inertial_cylinder mass="0.1" length="0.04" radius="0.05">
+            <origin xyz="0.0 0.0 0.0" rpy="0.0 0.0 0.0"/>
+        </xacro:inertial_cylinder>
+    </link>
+    <gazebo reference="left_wheel">
+        <material>Gazebo/Black</material>
+    </gazebo>
+    <!-- RIGHT WHEEL -->
+    <joint name="right_wheel_joint" type="continuous">
+        <origin xyz="0.0 -0.175 0.0" rpy="${pi/2} 0.0 0.0"/>
+        <parent link="base_link"/>
+        <child link="right_wheel"/>
+        <axis xyz="0.0 0.0 -1.0"/>
+    </joint>
+    <link name="right_wheel">
+        <visual>
+            <geometry>
+                <cylinder radius="0.05" length="0.04"/>
+            </geometry>
+            <material name="black"/>
+        </visual>
+        <collision>
+            <geometry>
+                <cylinder radius="0.05" length="0.04"/>
+            </geometry>
+        </collision>
+        <xacro:inertial_cylinder mass="0.1" length="0.04" radius="0.05">
+            <origin xyz="0.0 0.0 0.0" rpy="0.0 0.0 0.0"/>
+        </xacro:inertial_cylinder>
+    </link>
+    <gazebo reference="right_wheel">
+        <material>Gazebo/Black</material>
+    </gazebo>
+    <!-- CASTER WHEEL -->
+    <joint name="caster_wheel_joint" type="fixed">
+        <origin xyz="0.075 0.0 0.0"/>
+        <parent link="chassis"/>
+        <child link="caster_wheel"/>
+    </joint>
+    <link name="caster_wheel">
+        <visual>
+            <geometry>
+                <sphere radius="0.05"/>
+            </geometry>
+            <material name="black"/>
+        </visual>
+        <collision>
+            <geometry>
+                <sphere radius="0.05"/>
+            </geometry>
+        </collision>
+        <xacro:inertial_sphere mass="0.5" radius="0.05">
+            <origin xyz="0.0 0.0 0.0" rpy="0.0 0.0 0.0"/>
+        </xacro:inertial_sphere>
+    </link>
+    <gazebo reference="caster_wheel">
+        <material>Gazebo/Black</material>
+        <mu1 value="0.001"/>
+        <mu2 value="0.001"/>
+    </gazebo>
 </robot>
