Commit message: Added ros2_control to simulation. Updated URDF.

File: description/camera.xacro (robot description, xacro)
@@ -2,5 +2,5 @@
 <robot xmlns:xacro="http://www.ros.org/wiki/xacro">
     <joint name="camera_joint" type="fixed">
-        <origin xyz="0.305 0.0 0.05" rpy="0.0 0.0 0.0"/>
+        <origin xyz="0.202 0.0 ${chassis_height/2}" rpy="0.0 0.0 0.0"/>
         <parent link="chassis"/>
         <child link="camera"/>
@@ -9,5 +9,5 @@
         <visual>
             <geometry>
-                <box size="0.010 0.03 0.03"/>
+                <box size="0.002 0.03 0.03"/>
             </geometry>
             <material name="red"/>

File: description/lidar.xacro (robot description, xacro)
@@ -2,5 +2,5 @@
 <robot xmlns:xacro="http://www.ros.org/wiki/xacro">
     <joint name="lidar_joint" type="fixed">
-        <origin xyz="0.15 0.0 0.12" rpy="0.0 0.0 0.0"/>
+        <origin xyz="0.085 0.0 0.075" rpy="0.0 0.0 0.0"/>
         <parent link="chassis"/>
         <child link="lidar"/>
@@ -9,19 +9,19 @@
         <visual>
             <geometry>
-                <cylinder radius="0.05" length="0.04"/>
+                <cylinder radius="0.035" length="0.05"/>
             </geometry>
-            <material name="red"/>
+            <material name="black"/>
         </visual>
         <collision>
             <geometry>
-                <cylinder radius="0.05" length="0.04"/>
+                <cylinder radius="0.035" length="0.05"/>
             </geometry>
         </collision>
-        <xacro:inertial_cylinder mass="0.1" length="0.04" radius="0.05">
+        <xacro:inertial_cylinder mass="0.1" length="0.05" radius="0.035">
             <origin xyz="0.0 0.0 0.0" rpy="0.0 0.0 0.0"/>
         </xacro:inertial_cylinder>
     </link>
     <gazebo reference="lidar">
-        <material>Gazebo/Red</material>
+        <material>Gazebo/Black</material>
         <sensor name="lidar" type="ray">
             <pose> 0 0 0 0 0 0 </pose>

File: description/robot.urdf.xacro (robot description, xacro)
@@ -1,7 +1,15 @@
 <?xml version="1.0"?>
 <robot xmlns:xacro="http://www.ros.org/wiki/xacro" name="robot">
+    <xacro:arg name="use_ros2_control" default="true"/>
+    <xacro:include filename="parameters.xacro"/>
     <xacro:include filename="inertial_macros.xacro"/>
     <xacro:include filename="robot_core.xacro"/>
-    <xacro:include filename="gazebo_control.xacro"/>
+    <!-- Select between ros2_control or gazebo_control -->
+    <xacro:if value="$(arg use_ros2_control)">
+        <xacro:include filename="ros2_control.xacro"/>
+    </xacro:if>
+    <xacro:unless value="$(arg use_ros2_control)">
+        <xacro:include filename="gazebo_control.xacro"/>
+    </xacro:unless>
     <xacro:include filename="lidar.xacro"/>
     <xacro:include filename="camera.xacro"/>

File: description/robot_core.xacro (robot description, xacro)
@@ -9,31 +9,31 @@
         <parent link="base_link"/>
         <child link="chassis"/>
-        <origin xyz="-0.15 0.0 0.0"/>
+        <origin xyz="${-wheel_offset_x} 0.0 ${wheel_offset_z}"/>
     </joint>
     <link name="chassis">
         <visual>
             <!-- origin offset (review robot dimensions) -->
-            <origin xyz="0.15 0.0 0.05"/>
+            <origin xyz="${chassis_diameter/2} 0.0 ${chassis_height/2}"/>
             <geometry>
-                <cylinder radius="0.15" length="0.10"/>
+                <cylinder radius="${chassis_diameter/2}" length="${chassis_height}"/>
             </geometry>
-            <material name="gray"/>
+            <material name="white"/>
         </visual>
         <collision>
-            <origin xyz="0.15 0.0 0.05"/>
+            <origin xyz="${chassis_diameter/2} 0.0 ${chassis_height/2}"/>
             <geometry>
-                <cylinder radius="0.15" length="0.1"/>
+                <cylinder radius="${chassis_diameter/2}" length="${chassis_height}"/>
             </geometry>
         </collision>
-        <xacro:inertial_cylinder mass="0.5" length="0.1" radius="0.15">
-            <origin xyz="0.15 0.0 0.05" rpy="0.0 0.0 0.0"/>
+        <xacro:inertial_cylinder mass="${chassis_mass}" length="${chassis_height}" radius="${chassis_diameter/2}">
+            <origin xyz="${chassis_diameter/2} 0.0 ${chassis_height/2}" rpy="0.0 0.0 0.0"/>
         </xacro:inertial_cylinder>
     </link>
     <gazebo reference="chassis">
-        <material>Gazebo/LightGray</material>
+        <material>Gazebo/White</material>
     </gazebo>
     <!-- LEFT WHEEL -->
     <joint name="left_wheel_joint" type="continuous">
-        <origin xyz="0.0 0.175 0.0" rpy="-${pi/2} 0.0 0.0"/>
+        <origin xyz="0.0 ${wheel_offset_y} 0.0" rpy="-${pi/2} 0.0 0.0"/>
         <parent link="base_link"/>
         <child link="left_wheel"/>
@@ -43,23 +43,23 @@
         <visual>
             <geometry>
-                <cylinder radius="0.05" length="0.04"/>
+                <cylinder radius="${wheel_radius}" length="${wheel_thickness}"/>
             </geometry>
-            <material name="black"/>
+            <material name="blue"/>
         </visual>
         <collision>
             <geometry>
-                <cylinder radius="0.05" length="0.04"/>
+                <cylinder radius="${wheel_radius}" length="${wheel_thickness}"/>
             </geometry>
         </collision>
-        <xacro:inertial_cylinder mass="0.1" length="0.04" radius="0.05">
+        <xacro:inertial_cylinder mass="${wheel_mass}" length="${wheel_thickness}" radius="${wheel_radius}">
             <origin xyz="0.0 0.0 0.0" rpy="0.0 0.0 0.0"/>
         </xacro:inertial_cylinder>
     </link>
     <gazebo reference="left_wheel">
-        <material>Gazebo/Black</material>
+        <material>Gazebo/Blue</material>
     </gazebo>
     <!-- RIGHT WHEEL -->
     <joint name="right_wheel_joint" type="continuous">
-        <origin xyz="0.0 -0.175 0.0" rpy="${pi/2} 0.0 0.0"/>
+        <origin xyz="0.0 ${-wheel_offset_y} 0.0" rpy="${pi/2} 0.0 0.0"/>
         <parent link="base_link"/>
         <child link="right_wheel"/>
@@ -69,23 +69,23 @@
         <visual>
             <geometry>
-                <cylinder radius="0.05" length="0.04"/>
+                <cylinder radius="${wheel_radius}" length="${wheel_thickness}"/>
             </geometry>
-            <material name="black"/>
+            <material name="blue"/>
         </visual>
         <collision>
             <geometry>
-                <cylinder radius="0.05" length="0.04"/>
+                <cylinder radius="${wheel_radius}" length="${wheel_thickness}"/>
             </geometry>
         </collision>
-        <xacro:inertial_cylinder mass="0.1" length="0.04" radius="0.05">
+        <xacro:inertial_cylinder mass="${wheel_mass}" length="${wheel_thickness}" radius="${wheel_radius}">
             <origin xyz="0.0 0.0 0.0" rpy="0.0 0.0 0.0"/>
         </xacro:inertial_cylinder>
     </link>
     <gazebo reference="right_wheel">
-        <material>Gazebo/Black</material>
+        <material>Gazebo/Blue</material>
     </gazebo>
     <!-- CASTER WHEEL -->
     <joint name="caster_wheel_joint" type="fixed">
-        <origin xyz="0.075 0.0 0.0"/>
+        <origin xyz="${caster_wheel_offset_x} 0.0 ${-caster_wheel_offset_z}"/>
         <parent link="chassis"/>
         <child link="caster_wheel"/>
@@ -94,5 +94,5 @@
         <visual>
             <geometry>
-                <sphere radius="0.05"/>
+                <sphere radius="${caster_wheel_radius}"/>
             </geometry>
             <material name="black"/>
@@ -100,8 +100,8 @@
         <collision>
             <geometry>
-                <sphere radius="0.05"/>
+                <sphere radius="${caster_wheel_radius}"/>
             </geometry>
         </collision>
-        <xacro:inertial_sphere mass="0.5" radius="0.05">
+        <xacro:inertial_sphere mass="${caster_wheel_mass}" radius="${caster_wheel_radius}">
             <origin xyz="0.0 0.0 0.0" rpy="0.0 0.0 0.0"/>
         </xacro:inertial_sphere>
