Commit message: Added robot visuals in Gazebo

File: description/robot_core.xacro (robot description, xacro)
@@ -30,4 +30,7 @@
 		</xacro:inertial_cylinder>
 	</link>
+	<gazebo reference="chassis">
+		<material>Gazebo/LightGray</material>
+	</gazebo>
 	<!-- LEFT WHEEL -->
 	<joint name="left_wheel_joint" type="continuous">
@@ -53,4 +56,7 @@
 		</xacro:inertial_cylinder>
 	</link>
+	<gazebo reference="left_wheel">
+		<material>Gazebo/Black</material>
+	</gazebo>
 	<!-- RIGHT WHEEL -->
 	<joint name="right_wheel_joint" type="continuous">
@@ -76,4 +82,7 @@
 		</xacro:inertial_cylinder>
 	</link>
+	<gazebo reference="right_wheel">
+		<material>Gazebo/Black</material>
+	</gazebo>
 	<!-- CASTER WHEEL -->
 	<joint name="caster_wheel_joint" type="fixed">
@@ -98,3 +107,6 @@
 		</xacro:inertial_sphere>
 	</link>
+	<gazebo reference="caster_wheel">
+		<material>Gazebo/Black</material>
+	</gazebo>
 </robot>

Commit message: Added slam_toolbox.

File: description/robot_core.xacro (robot description, xacro)
@@ -4,4 +4,12 @@
     <!-- BASE LINK -->
     <link name="base_link">
+    </link>
+    <!-- BASE FOOTPRINT LINK -->
+    <joint name="base_footprint_joint" type="fixed">
+        <parent link="base_link"/>
+        <child link="base_footprint"/>
+        <origin xyz="0.0 0.0 0.0" rpy="0.0 0.0 0.0"/>
+    </joint>
+    <link name="base_footprint">
     </link>
     <!-- CHASSIS -->
